File: nixie3.kicad_sch (KiCad schematic)
At the start: 50 parts, among them J1 AVR-ISP-10, J2 Barrel_Jack, J3 Conn_01x02_Pin, J4 Conn_01x02_Pin, J5 Conn_01x02_Pin, J6 Conn_01x02_Pin, J7 Conn_01x02_Pin, J8 Conn_01x02_Pin, Q1 IRFB4020PBF, U1 ATmega328-A, U2 MCP1401T-E/OT, U3 HV5222PG-G, U4 HV5222PG-G, U5 MC34063AP, X1 CXO_DIP8

Commit message: Updates.
Parts:
- removed J1: AVR-ISP-10, Connector_PinHeader_2.54mm:PinHeader_2x05_P2.54mm_Vertical, symbol Connector:AVR-ISP-10
- removed J3, J4: Conn_01x02_Pin, Connector_PinHeader_2.54mm:PinHeader_1x02_P2.54mm_Vertical, symbol Connector:Conn_01x02_Pin
- removed X1: CXO_DIP8, Oscillator:Oscillator_DIP-8, symbol Oscillator:CXO_DIP8
- added C10, C11, C14: 100nF, symbol Device:C
- added C12: 10uF, symbol Device:C_Polarized
- added C13: 100uF 25V, symbol Device:C_Polarized
- added C6: 12pF, Capacitor_THT:C_Disc_D5.0mm_W2.5mm_P5.00mm, symbol Device:C
- added C7: 18pF, Capacitor_THT:C_Disc_D5.0mm_W2.5mm_P5.00mm, symbol Device:C
- added C8, C9: 47pF, symbol Device:C
- added J1: USB_B, symbol Connector:USB_B
- added J9: AVR-ISP-6, Connector_PinHeader_2.54mm:PinHeader_2x03_P2.54mm_Vertical, symbol Connector:AVR-ISP-6
- added R17: 10k, Resistor_THT:R_Axial_DIN0207_L6.3mm_D2.5mm_P2.54mm_Vertical, symbol Device:R_US
- added R18, R19: 27, symbol Device:R_US
- added U6: FT231XS-R, FT231XS-R:SOP63P599X175-20N, symbol ftdi:FT231XS-R
- added U7: CD40109BNSR, NS16, symbol cd40109:CD40109BNSR
- added Y1: 10MHz / 12pF, Crystal:Crystal_HC49-U_Vertical, symbol Device:Crystal
- C3: value C -> 10uF 400V
- J2: value Barrel_Jack -> 12V PWR
- U3, U4: footprint import1:QFP44_10x10MC_MCH -> import1:QFP44_10x10MC_MCH-M
Connections:
- net GND: now also C10.2, C11.2, C12.2, C13.2, C14.2, C6.1, C7.1, C8.2, C9.2, J1.4 (GND), J1.5 (Shield), J9.6 (GND), U6.16 (GND), U6.6 (GND), U6.7 (~{DSR}), U6.8 (~{DCD}), U6.9 (~{CTS}), U7.8 (VSS)
- net VCC: now also C13.1, C14.1, U7.16 (VDD)
- net VDD: now also C10.1, C11.1, C12.1, J9.2 (VCC), R17.2, U6.14 (~{RESET}), U6.15 (VCC), U6.3 (VCCIO), U7.1 (VCC), U7.15 (ENABLED), U7.2 (ENABLEA), U7.7 (ENABLEB), U7.9 (ENABLEC)
- net at U1.10 (PD6), U2.3 (IN): now also R17.1
- net at U1.11 (PD7): now also J5.1 (Pin_1)
- net at U1.15 (PB3): now also J9.4 (MOSI)
- net at U1.16 (PB4): now also J9.1 (MISO)
- net at U1.17 (PB5): now also J9.3 (SCK)
- net at U3.32 (STR), U4.32 (STR): now also U7.11 (G); no longer U1.25 (PC2)
- net at U1.26 (PC3): now also U7.14 (D)
- net at U1.27 (PC4): now also U7.3 (A)
- net at U3.29 (CLK), U4.29 (CLK): now also U7.5 (F); no longer U1.28 (PC5)
- net at C1.1, R1.2, U1.29 (~{RESET}/PC6): now also J9.5 (~{RST})
- net at U1.30 (PD0): now also U6.20 (TXD)
- net at U1.31 (PD1): now also U6.4 (RXD)
- net at U1.32 (PD2): now also U6.2 (~{RTS}); no longer J5.1 (Pin_1)
- net at U1.7 (XTAL1/PB6): now also C7.2, Y1.2
- net at U1.8 (XTAL2/PB7): now also C6.2, Y1.1
- net at U3.28 (OE), U4.28 (OE): now also U7.13 (H)
- net at U3.33 (DATAIN): now also U7.4 (E)
- new net: U1.25 (PC2), U7.10 (C)
- new net: U1.28 (PC5), U7.6 (B)
- new net: R18.1, U6.11 (USBDP)
- new net: C9.1, J1.3 (D+), R18.2
- new net: R19.1, U6.12 (USBDM)
- new net: C8.1, J1.2 (D-), R19.2
Other:
- moved on the sheet: NE1, NE2, NE3, NE4, NX1, NX2, NX3, NX4, NX5, NX6, R10, R11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

Commit message: Updates.
Parts:
- removed U3, U4: HV5222PG-G, import1:QFP44_10x10MC_MCH-M, symbol import1:HV5222PG-G
- removed U7: CD40109BNSR, NS16, symbol cd40109:CD40109BNSR
- added U10, U11, U12, U7, U8, U9: 74141, Package_DIP:DIP-16_W7.62mm, symbol 74xx_IEEE:74141
- added U13: 74AHC595, Package_DIP:DIP-16_W7.62mm, symbol 74xx:74AHC595
- added U14, U15: 74HC595, Package_DIP:DIP-16_W7.62mm, symbol 74xx:74HC595
- C10, C11, C12, C14, C8, C9: footprint (none) -> Capacitor_THT:CP_Radial_D5.0mm_P2.50mm
- C13: footprint (none) -> Capacitor_THT:CP_Radial_D8.0mm_P5.00mm
- J1: footprint (none) -> Connector_USB:USB_B_OST_USB-B1HSxx_Horizontal
- R18, R19: footprint (none) -> Resistor_THT:R_Axial_DIN0204_L3.6mm_D1.6mm_P2.54mm_Vertical
- U6: footprint FT231XS-R:SOP63P599X175-20N -> import3:SOP63P599X175-20N
Connections:
- net Net-(U3A-HVOUT1) is gone; now on net GND: NE2.2
- net Net-(U3A-HVOUT12) is gone; now on net GND: NE1.2
- net unconnected-(U4A-HVOUT21-Pad2) is gone; now on net GND: NE4.2
- net unconnected-(U4A-HVOUT22-Pad1) is gone; now on net GND: NE3.2
- net GND: now also U13.13 (~{OE}), U13.8 (GND), U14.13 (~{OE}), U14.8 (GND), U15.13 (~{OE}), U15.8 (GND)
- net VDD: now also U13.10 (~{SRCLR}), U13.16 (VCC), U14.10 (~{SRCLR}), U14.16 (VCC), U15.10 (~{SRCLR}), U15.16 (VCC)
- net at J7.1 (Pin_1): now also U1.25 (PC2); no longer U1.2 (PD4)
- net at U1.1 (PD3): now also U13.12 (RCLK), U14.12 (RCLK), U15.12 (RCLK); no longer J6.1 (Pin_1)
- net at R17.1, U2.3 (IN): now also U1.9 (PD5); no longer U1.10 (PD6)
- net at U1.11 (PD7): no longer J5.1 (Pin_1)
- net at U1.23 (PC0): now also J5.1 (Pin_1)
- net at U1.24 (PC1): now also J6.1 (Pin_1)
- net at U1.26 (PC3): now also J8.1 (Pin_1)
- net at U1.27 (PC4): now also U13.14 (SER)
- net at U1.28 (PC5): now also U13.11 (SRCLK), U14.11 (SRCLK), U15.11 (SRCLK)
- net Net-(U3A-HVOUT10): no longer names the net of NX3.6
- net Net-(U3A-HVOUT10): now also U11.11 (~{Q6})
- net Net-(U3A-HVOUT11): no longer names the net of NX3.5
- net Net-(U3A-HVOUT11): now also U11.14 (~{Q5})
- net Net-(U3A-HVOUT13): no longer names the net of NX2.0
- net Net-(U3A-HVOUT13): now also U10.16 (~{Q0})
- net Net-(U3A-HVOUT14): no longer names the net of NX2.9
- net Net-(U3A-HVOUT14): now also U10.2 (~{Q9})
- net Net-(U3A-HVOUT15): no longer names the net of NX2.8
- net Net-(U3A-HVOUT15): now also U10.1 (~{Q8})
- net Net-(U3A-HVOUT16): no longer names the net of NX2.7
- net Net-(U3A-HVOUT16): now also U10.10 (~{Q7})
- net Net-(U3A-HVOUT17): no longer names the net of NX2.6
- net Net-(U3A-HVOUT17): now also U10.11 (~{Q6})
- net Net-(U3A-HVOUT18): no longer names the net of NX2.5
- net Net-(U3A-HVOUT18): now also U10.14 (~{Q5})
- net Net-(U3A-HVOUT19): no longer names the net of NX2.4
- net Net-(U3A-HVOUT19): now also U10.13 (~{Q4})
- net Net-(U3A-HVOUT2): no longer names the net of NX3.4
- net Net-(U3A-HVOUT2): now also U11.13 (~{Q4})
- net Net-(U3A-HVOUT20): no longer names the net of NX2.3
- net Net-(U3A-HVOUT20): now also U10.9 (~{Q3})
- net Net-(U3A-HVOUT21): no longer names the net of NX2.2
- net Net-(U3A-HVOUT21): now also U10.8 (~{Q2})
- net Net-(U3A-HVOUT22): no longer names the net of NX2.1
- net Net-(U3A-HVOUT22): now also U10.15 (~{Q1})
- net Net-(U3A-HVOUT23): no longer names the net of NX1.0
- net Net-(U3A-HVOUT23): now also U8.16 (~{Q0})
- net Net-(U3A-HVOUT24): no longer names the net of NX1.9
- net Net-(U3A-HVOUT24): now also U8.2 (~{Q9})
- net Net-(U3A-HVOUT25): no longer names the net of NX1.8
- net Net-(U3A-HVOUT25): now also U8.1 (~{Q8})
- net Net-(U3A-HVOUT26): no longer names the net of NX1.7
- net Net-(U3A-HVOUT26): now also U8.10 (~{Q7})
- net Net-(U3A-HVOUT27): no longer names the net of NX1.6
- net Net-(U3A-HVOUT27): now also U8.11 (~{Q6})
- net Net-(U3A-HVOUT28): no longer names the net of NX1.5
- net Net-(U3A-HVOUT28): now also U8.14 (~{Q5})
- net Net-(U3A-HVOUT29): no longer names the net of NX1.4
- net Net-(U3A-HVOUT29): now also U8.13 (~{Q4})
- net Net-(U3A-HVOUT3): no longer names the net of NX3.3
- net Net-(U3A-HVOUT3): now also U11.9 (~{Q3})
- net Net-(U3A-HVOUT30): no longer names the net of NX1.3
- net Net-(U3A-HVOUT30): now also U8.9 (~{Q3})
- net Net-(U3A-HVOUT31): no longer names the net of NX1.2
- net Net-(U3A-HVOUT31): now also U8.8 (~{Q2})
- net Net-(U3A-HVOUT32): no longer names the net of NX1.1
- net Net-(U3A-HVOUT32): now also U8.15 (~{Q1})
- net Net-(U3A-HVOUT4): no longer names the net of NX3.2
- net Net-(U3A-HVOUT4): now also U11.8 (~{Q2})
- net Net-(U3A-HVOUT5): no longer names the net of NX3.1
- net Net-(U3A-HVOUT5): now also U11.15 (~{Q1})
- net Net-(U3A-HVOUT6): no longer names the net of NX3.0
- net Net-(U3A-HVOUT6): now also U11.16 (~{Q0})
- net Net-(U3A-HVOUT7): no longer names the net of NX3.9
- net Net-(U3A-HVOUT7): now also U11.2 (~{Q9})
- net Net-(U3A-HVOUT8): no longer names the net of NX3.8
- net Net-(U3A-HVOUT8): now also U11.1 (~{Q8})
- net Net-(U3A-HVOUT9): no longer names the net of NX3.7
- net Net-(U3A-HVOUT9): now also U11.10 (~{Q7})
- net unconnected-(U4A-HVOUT1-Pad22): no longer names the net of NX6.0
- net unconnected-(U4A-HVOUT1-Pad22): now also U12.16 (~{Q0})
- net unconnected-(U4A-HVOUT10-Pad13): no longer names the net of NX6.1
- net unconnected-(U4A-HVOUT10-Pad13): now also U12.15 (~{Q1})
- net unconnected-(U4A-HVOUT11-Pad12): no longer names the net of NX5.0
- net unconnected-(U4A-HVOUT11-Pad12): now also U9.16 (~{Q0})
- net unconnected-(U4A-HVOUT12-Pad11): no longer names the net of NX5.9
- net unconnected-(U4A-HVOUT12-Pad11): now also U9.2 (~{Q9})
- net unconnected-(U4A-HVOUT13-Pad10): no longer names the net of NX5.8
- net unconnected-(U4A-HVOUT13-Pad10): now also U9.1 (~{Q8})
- net unconnected-(U4A-HVOUT14-Pad9): no longer names the net of NX5.7
- net unconnected-(U4A-HVOUT14-Pad9): now also U9.10 (~{Q7})
- net unconnected-(U4A-HVOUT15-Pad8): no longer names the net of NX5.6
- net unconnected-(U4A-HVOUT15-Pad8): now also U9.11 (~{Q6})
- net unconnected-(U4A-HVOUT16-Pad7): no longer names the net of NX5.5
- net unconnected-(U4A-HVOUT16-Pad7): now also U9.14 (~{Q5})
- net unconnected-(U4A-HVOUT17-Pad6): no longer names the net of NX5.4
- net unconnected-(U4A-HVOUT17-Pad6): now also U9.13 (~{Q4})
- net unconnected-(U4A-HVOUT18-Pad5): no longer names the net of NX5.3
- net unconnected-(U4A-HVOUT18-Pad5): now also U9.9 (~{Q3})
- net unconnected-(U4A-HVOUT19-Pad4): no longer names the net of NX5.2
- net unconnected-(U4A-HVOUT19-Pad4): now also U9.8 (~{Q2})
- net unconnected-(U4A-HVOUT2-Pad21): no longer names the net of NX6.9
- net unconnected-(U4A-HVOUT2-Pad21): now also U12.2 (~{Q9})
- net unconnected-(U4A-HVOUT20-Pad3): no longer names the net of NX5.1
- net unconnected-(U4A-HVOUT20-Pad3): now also U9.15 (~{Q1})
- net unconnected-(U4A-HVOUT23-Pad44): no longer names the net of NX4.0
- net unconnected-(U4A-HVOUT23-Pad44): now also U7.16 (~{Q0})
- net unconnected-(U4A-HVOUT24-Pad43): no longer names the net of NX4.9
- net unconnected-(U4A-HVOUT24-Pad43): now also U7.2 (~{Q9})
- net unconnected-(U4A-HVOUT25-Pad42): no longer names the net of NX4.8
- net unconnected-(U4A-HVOUT25-Pad42): now also U7.1 (~{Q8})
- net unconnected-(U4A-HVOUT26-Pad41): no longer names the net of NX4.7
- net unconnected-(U4A-HVOUT26-Pad41): now also U7.10 (~{Q7})
- net unconnected-(U4A-HVOUT27-Pad40): no longer names the net of NX4.6
- net unconnected-(U4A-HVOUT27-Pad40): now also U7.11 (~{Q6})
- net unconnected-(U4A-HVOUT28-Pad39): no longer names the net of NX4.5
- net unconnected-(U4A-HVOUT28-Pad39): now also U7.14 (~{Q5})
- net unconnected-(U4A-HVOUT29-Pad38): no longer names the net of NX4.4
- net unconnected-(U4A-HVOUT29-Pad38): now also U7.13 (~{Q4})
- net unconnected-(U4A-HVOUT3-Pad20): no longer names the net of NX6.8
- net unconnected-(U4A-HVOUT3-Pad20): now also U12.1 (~{Q8})
- net unconnected-(U4A-HVOUT30-Pad37): no longer names the net of NX4.3
- net unconnected-(U4A-HVOUT30-Pad37): now also U7.9 (~{Q3})
- net unconnected-(U4A-HVOUT31-Pad36): no longer names the net of NX4.2
- net unconnected-(U4A-HVOUT31-Pad36): now also U7.8 (~{Q2})
- net unconnected-(U4A-HVOUT32-Pad35): no longer names the net of NX4.1
- net unconnected-(U4A-HVOUT32-Pad35): now also U7.15 (~{Q1})
- net unconnected-(U4A-HVOUT4-Pad19): no longer names the net of NX6.7
- net unconnected-(U4A-HVOUT4-Pad19): now also U12.10 (~{Q7})
- net unconnected-(U4A-HVOUT5-Pad18): no longer names the net of NX6.6
- net unconnected-(U4A-HVOUT5-Pad18): now also U12.11 (~{Q6})
- net unconnected-(U4A-HVOUT6-Pad17): no longer names the net of NX6.5
- net unconnected-(U4A-HVOUT6-Pad17): now also U12.14 (~{Q5})
- net unconnected-(U4A-HVOUT7-Pad16): no longer names the net of NX6.4
- net unconnected-(U4A-HVOUT7-Pad16): now also U12.13 (~{Q4})
- net unconnected-(U4A-HVOUT8-Pad15): no longer names the net of NX6.3
- net unconnected-(U4A-HVOUT8-Pad15): now also U12.9 (~{Q3})
- net unconnected-(U4A-HVOUT9-Pad14): no longer names the net of NX6.2
- net unconnected-(U4A-HVOUT9-Pad14): now also U12.8 (~{Q2})
- new net: U14.4 (QE), U7.3 (A)
- new net: U14.7 (QH), U7.4 (D)
- new net: U14.5 (QF), U7.6 (B)
- new net: U14.6 (QG), U7.7 (C)
- new net: U15.15 (QA), U9.3 (A)
- new net: U15.3 (QD), U9.4 (D)
- new net: U15.1 (QB), U9.6 (B)
- new net: U15.2 (QC), U9.7 (C)
- new net: U13.15 (QA), U8.3 (A)
- new net: U13.3 (QD), U8.4 (D)
- new net: U13.1 (QB), U8.6 (B)
- new net: U13.2 (QC), U8.7 (C)
- new net: U11.6 (B), U14.1 (QB)
- new net: U13.9 (QH'), U14.14 (SER)
- new net: U11.3 (A), U14.15 (QA)
- new net: U11.7 (C), U14.2 (QC)
- new net: U11.4 (D), U14.3 (QD)
- new net: U14.9 (QH'), U15.14 (SER)
- new net: U10.3 (A), U13.4 (QE)
- new net: U10.6 (B), U13.5 (QF)
- new net: U10.7 (C), U13.6 (QG)
- new net: U10.4 (D), U13.7 (QH)
- new net: U12.3 (A), U15.4 (QE)
- new net: U12.6 (B), U15.5 (QF)
- new net: U12.7 (C), U15.6 (QG)
- new net: U12.4 (D), U15.7 (QH)

Commit message: board update
Connections:
- net GND: now also U10.12 (GND), U11.12 (GND), U12.12 (GND), U7.12 (GND), U8.12 (GND), U9.12 (GND)
- net VDD: now also U10.5 (VCC), U11.5 (VCC), U12.5 (VCC), U7.5 (VCC), U8.5 (VCC), U9.5 (VCC)

Commit message: final board layout.
Connections:
- net at U1.13 (PB1): now also R17.1, U2.3 (IN)
- now unconnected: U1.9 (PD5)
Changed lines of the file:
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@@
-    (stroke (width 0) (type default))
-  )
-  (wire (pts (xy 109.22 137.16) (xy 109.22 211.455))
     (stroke (width 0) (type default))
   )
@@
     (stroke (width 0) (type default))
   )
+  (wire (pts (xy 109.22 83.82) (xy 109.22 211.455))
+    (stroke (width 0) (type default))
+  )
   (wire (pts (xy 276.225 313.055) (xy 276.225 250.825))
     (stroke (width 0) (type default))
@@
     (stroke (width 0) (type default))
   )
+  (wire (pts (xy 109.22 83.82) (xy 95.25 83.82))
+    (stroke (width 0) (type default))
+  )
   (wire (pts (xy 342.9 259.715) (xy 372.745 259.715))
     (stroke (width 0) (type default))
@@
     (stroke (width 0) (type default))
   )
-  (wire (pts (xy 95.25 137.16) (xy 109.22 137.16))
-    (stroke (width 0) (type default))
-  )
